Commit message: Correct wheel_radius to measured 0.30m (was 0.15m placeholder)
실측 결과 구동륜 반지름은 0.30m. urdf.xacro와 base_driver.py 양쪽 기본값을
수정. lidar_z는 base_link 기준 상대값(0.35)이라 그대로 두었고, 라이다의
지면 기준 실제 높이는 wheel_radius + lidar_z = 0.65m로 자동 반영됨.

Co-Authored-By: Claude Sonnet 5 <noreply@anthropic.com>
Claude-Session: https://claude.ai/code/session_01Aw8oJxPZSDBbGUorkNB2C6

File: src/autonomous_wheelchair/urdf/wheelchair.urdf.xacro (robot description, xacro)
@@ -5,5 +5,5 @@
   <xacro:property name="chassis_width" value="0.70"/>
   <xacro:property name="chassis_height" value="0.40"/>
-  <xacro:property name="wheel_radius" value="0.15"/>
+  <xacro:property name="wheel_radius" value="0.30"/>
   <xacro:property name="wheel_width" value="0.05"/>
   <xacro:property name="wheel_separation" value="0.56"/>

Commit message: Update lidar mount height to actual 0.50m (lidar_z 0.35 -> 0.20)
실제로 라이다를 지면 기준 0.50m 높이에 장착. base_link가 wheel_radius
(0.30m)만큼 지면에서 떠 있으므로 base_link 기준 상대값은 0.50-0.30=0.20.

Co-Authored-By: Claude Sonnet 5 <noreply@anthropic.com>
Claude-Session: https://claude.ai/code/session_01Aw8oJxPZSDBbGUorkNB2C6

File: src/autonomous_wheelchair/urdf/wheelchair.urdf.xacro (robot description, xacro)
@@ -12,5 +12,5 @@
   <xacro:property name="lidar_x" value="0.55"/>
   <xacro:property name="lidar_y" value="0.0"/>
-  <xacro:property name="lidar_z" value="0.35"/>
+  <xacro:property name="lidar_z" value="0.20"/>
   <material name="grey">
     <color rgba="0.5 0.5 0.5 1.0"/>
